File: OpenPSX2AmigaPadAdapter.sch (KiCad schematic (older format))
At the start: 44 parts, among them J1 TO_PSX_PAD, J2 DB9_F, J3 CONN_FTDI, J4 CONN_ICSP, J99 OSHW_LOGO, Q1 BSS138, Q2 BSS138, Q3 BSS138, Q4 BSS138, Q5 BSS138, SW1 RESET, U1 ATmega328P-AU, U2 LM1117-3.3, Y1 16M, Y2 16M

Commit message: Update schematics for analog output support. PCB TBD.
Parts:
- removed SW1: RESET, symbol Switch:SW_Push
- removed U2: LM1117-3.3, Package_TO_SOT_SMD:SOT-223-3_TabPin2, symbol Regulator_Linear:LM1117-3.3
- added R17: 10k, Resistor_SMD:R_0805_2012Metric_Pad1.15x1.40mm_HandSolder, symbol Device:R
- added R18, R19: 1M, Resistor_SMD:R_0805_2012Metric_Pad1.15x1.40mm_HandSolder, symbol Device:R
- added U2: TC1185-3.3V, Package_TO_SOT_SMD:SOT-23-5_HandSoldering, symbol Regulator_Linear:TC1017-xCT
- added U3: AD5242, Package_SO:SOIC-16_3.9x9.9mm_P1.27mm, symbol ad5242:AD5242
- C1, C2: value 10u -> 1u; footprint Capacitor_SMD:C_1206_3216Metric_Pad1.42x1.75mm_HandSolder -> Capacitor_SMD:C_0805_2012Metric_Pad1.15x1.40mm_HandSolder
Connections:
- net labels added: scl, sda
- wire segments 201 -> 236
- no-connect marks 9 -> 10
Other:
- note added: "5V -> 3.3V\nUP to 150 mA"
- note added: "ANALOG OUTPUT\nGENERATION"
- note added: "DB-9 OUTPUT"
- note added: "DECOUPLING"
- note added: "LEVEL TRANSLATION"
- note added: "PROGRAMMING"
- note added: "PS2 INPUT"
- note added: "Resistance between Ax and Wx is:\n(256 − D) / 256 × Rab + Rw\n\nFor instance, with AD5242BR1M:\nRaw = 3966 ohm for D = 255\nRaw = 1000060 ohm for D = 0"
- note added: "STATUS LEDS"
- note added: "VOLTAGE REGULATION"
- note added: "When ~SHDN is asserted,\nTerminal A is open circuited\nand Wiper W is connected\nto Terminal B"
- note removed: "BOTH 10uF CAPS MUST\nPOSSIBLY BE TANTALUM"
- moved on the sheet: C10, C3, C4, C8, C9, D1, J1, J2, J3, J4, LD1, LD2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
